File: inf turret.kicad_pcb (KiCad board)
At the start: 2 copper layers, 45 x 45 mm, 27 parts, among them J1 Conn_01x06_Pin, J3 Conn_01x03_Pin, U1 XIAO-ESP32S3

Commit message: update the pcb a bit
Parts:
- removed C1: 0.1µF, Capacitor_SMD:C_0805_2012Metric
- C2: value 10µF -> 100µF
- moved C2 2.33 mm to (134.6, 99.4)
Routing:
- net GND: track 65.3 -> 52.5 mm
Changed lines of the file:
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@@
 	(footprint "Capacitor_SMD:C_1206_3216Metric"
 		(layer "F.Cu")
-		(at 133.4 101.4 180)
+		(at 134.6 99.4 180)
 		(descr "Capacitor SMD 1206 (3216 Metric), square (rectangular) end terminal, IPC_7351 nominal, (Body size source: IPC-SM-782 page 76, https://www.pcb-3d.com/wordpress/wp-content/uploads/ipc-sm-782a_amendment_1_and_2.pdf), generated with kicad-footprint-generator")
 		(tags "capacitor")
@@
 			)
 		)
-		(property "Value" "10µF"
+		(property "Value" "100µF"
 			(at 0 1.85 180)
 			(layer "F.Fab")
@@
 		(embedded_fonts no)
 	)
-	(footprint "Capacitor_SMD:C_0805_2012Metric"
-		(layer "F.Cu")
-		(at 133.8 98 180)
-		(descr "Capacitor SMD 0805 (2012 Metric), square (rectangular) end terminal, IPC_7351 nominal, (Body size source: IPC-SM-782 page 76, https://www.pcb-3d.com/wordpress/wp-content/uploads/ipc-sm-782a_amendment_1_and_2.pdf, https://docs.google.com/spreadsheets/d/1BsfQQcO9C6DZCsRaXUlFlo91Tg2WpOkGARC1WS5S8t0/edit?usp=sharing), generated with kicad-footprint-generator")
-		(tags "capacitor")
-		(property "Reference" "C1"
-			(at 0 -1.68 0)
-			(layer "F.SilkS")
-			(effects
-				(font
-					(size 1 1)
-					(thickness 0.15)
-				)
-			)
-		)
-		(property "Value" "0.1µF"
-			(at 0 1.68 0)
-			(layer "F.Fab")
-			(effects
-				(font
-					(size 1 1)
-					(thickness 0.15)
-				)
-			)
-		)
-		(property "Datasheet" "~"
-			(at 0 0 0)
-			(layer "F.Fab")
-			(hide yes)
-			(effects
-				(font
-					(size 1.27 1.27)
-					(thickness 0.15)
-				)
-			)
-		)
-		(property "Description" "Unpolarized capacitor"
-			(at 0 0 0)
-			(layer "F.Fab")
-			(hide yes)
-			(effects
-				(font
-					(size 1.27 1.27)
-					(thickness 0.15)
-				)
-			)
-		)
-		(property ki_fp_filters "C_*")
-		(sheetname "/")
-		(sheetfile "inf turret.kicad_sch")
-		(attr smd)
-		(fp_line
-			(start -0.261252 0.735)
-			(end 0.261252 0.735)
-			(stroke
-				(width 0.12)
-				(type solid)
-			)
-			(layer "F.SilkS")
-		)
-		(fp_line
-			(start -0.261252 -0.735)
-			(end 0.261252 -0.735)
-			(stroke
-				(width 0.12)
-				(type solid)
-			)
-			(layer "F.SilkS")
-		)
-		(fp_line
-			(start 1.7 0.98)
-			(end -1.7 0.98)
-			(stroke
-				(width 0.05)
-				(type solid)
-			)
-			(layer "F.CrtYd")
-		)
-		(fp_line
-			(start 1.7 -0.98)
-			(end 1.7 0.98)
-			(stroke
-				(width 0.05)
-				(type solid)
-			)
-			(layer "F.CrtYd")
-		)
-		(fp_line
-			(start -1.7 0.98)
-			(end -1.7 -0.98)
-			(stroke
-				(width 0.05)
-				(type solid)
-			)
-			(layer "F.CrtYd")
-		)
-		(fp_line
-			(start -1.7 -0.98)
-			(end 1.7 -0.98)
-			(stroke
-				(width 0.05)
-				(type solid)
-			)
-			(layer "F.CrtYd")
-		)
-		(fp_line
-			(start 1 0.625)
-			(end -1 0.625)
-			(stroke
-				(width 0.1)
-				(type solid)
-			)
-			(layer "F.Fab")
-		)
-		(fp_line
-			(start 1 -0.625)
-			(end 1 0.625)
-			(stroke
-				(width 0.1)
-				(type solid)
-			)
-			(layer "F.Fab")
-		)
-		(fp_line
-			(start -1 0.625)
-			(end -1 -0.625)
-			(stroke
-				(width 0.1)
-				(type solid)
-			)
-			(layer "F.Fab")
-		)
-		(fp_line
-			(start -1 -0.625)
-			(end 1 -0.625)
-			(stroke
-				(width 0.1)
-				(type solid)
-			)
-			(layer "F.Fab")
-		)
-		(fp_text user "${REFERENCE}"
-			(at 0 0 0)
-			(layer "F.Fab")
-			(effects
-				(font
-					(size 0.5 0.5)
-					(thickness 0.08)
-				)
-			)
-		)
-		(pad "1" smd roundrect
-			(at -0.95 0 180)
-			(size 1 1.45)
-			(layers "F.Cu" "F.Mask" "F.Paste")
-			(roundrect_rratio 0.25)
-			(net 1 "GND")
-			(pintype "passive")
-		)
-		(pad "2" smd roundrect
-			(at 0.95 0 180)
-			(size 1 1.45)
-			(layers "F.Cu" "F.Mask" "F.Paste")
-			(roundrect_rratio 0.25)
-			(net 2 "+5V")
-			(pintype "passive")
-		)
-		(embedded_fonts no)
-		(model "${KISYS3DMOD}/Capacitor_SMD.3dshapes/C_0805_2012Metric.wrl"
-			(offset
-				(xyz 0 0 0)
-			)
-			(scale
-				(xyz 1 1 1)
-			)
-			(rotate
-				(xyz 0 0 0)
-			)
-		)
-	)
 	(footprint ""
 		(layer "F.Cu")
@@
 	)
 	(segment
-		(start 140.15 92.6)
-		(end 143.52 92.6)
-		(width 0.2)
-		(layer "F.Cu")
-		(net 1)
-	)
-	(segment
-		(start 143.52 92.755)
-		(end 134.875 101.4)
-		(width 0.2)
-		(layer "F.Cu")
-		(net 1)
-	)
-	(segment
 		(start 128.173639 107.5)
 		(end 127.284768 108.388871)
@@
 	)
 	(segment
-		(start 134.75 98)
-		(end 140.15 92.6)
-		(width 0.2)
-		(layer "F.Cu")
-		(net 1)
-	)
-	(segment
 		(start 143.000001 81.198531)
 		(end 143 81.19853)
@@
 	)
 	(segment
-		(start 143.52 92.6)
-		(end 143.52 92.755)
-		(width 0.2)
-		(layer "F.Cu")
-		(net 1)
-	)
-	(segment
 		(start 130.506497 113.83198)
 		(end 130.506497 113.994841)
@@
 	)
 	(segment
-		(start 143.52 83.8)
-		(end 143.52 92.6)
+		(start 162.419238 88.419238)
+		(end 162.5 88.5)
 		(width 0.2)
 		(layer "F.Cu")
@@
 	)
 	(segment
-		(start 162.419238 88.419238)
-		(end 162.5 88.5)
+		(start 137.2 99.4)
+		(end 136.075 99.4)
 		(width 0.2)
 		(layer "F.Cu")
@@
 	)
 	(segment
+		(start 143.52 83.8)
+		(end 143.52 93.08)
+		(width 0.2)
+		(layer "F.Cu")
+		(net 1)
+	)
+	(segment
 		(start 164.652242 106.734634)
 		(end 164.652242 107.152242)
@@
 	)
 	(segment
+		(start 143.52 93.08)
+		(end 137.2 99.4)
+		(width 0.2)
+		(layer "F.Cu")
+		(net 1)
+	)
+	(segment
 		(start 128.652242 92.234634)
 		(end 127.500821 92.234634)
@@
 	)
 	(segment
-		(start 131.380172 96.819827)
-		(end 131.669827 96.819827)
-		(width 0.2)
-		(layer "F.Cu")
-		(net 2)
-	)
-	(segment
 		(start 167.999998 92.999998)
 		(end 167.03359 92.03359)
@@
 	(segment
 		(start 129.850269 99.85027)
-		(end 129.850269 101.2)
+		(end 129.850269 105.53359)
 		(width 0.5)
 		(layer "F.Cu")
@@
 	)
 	(segment
-		(start 129.850269 101.2)
-		(end 130.050269 101.4)
-		(width 0.2)
-		(layer "F.Cu")
-		(net 2)
-	)
-	(segment
 		(start 155.754161 80.35)
 		(end 152.499999 80.35)
@@
 	)
 	(segment
-		(start 130.050269 101.4)
-		(end 131.925 101.4)
-		(width 0.5)
-		(layer "F.Cu")
-		(net 2)
-	)
-	(segment
 		(start 147.5 120.5)
 		(end 147.5 117.5)
@@
 	)
 	(segment
-		(start 167.5 108.414213)
-		(end 164.166726 111.747487)
+		(start 132.850001 99.2)
+		(end 128.999999 99.2)
 		(width 0.5)
 		(layer "F.Cu")
@@
 	)
 	(segment
-		(start 166.997488 106.298956)
-		(end 167.5 106.801468)
+		(start 167.5 108.414213)
+		(end 164.166726 111.747487)
 		(width 0.5)
 		(layer "F.Cu")
@@
 	)
 	(segment
-		(start 129.850269 101.2)
-		(end 129.850269 105.53359)
+		(start 166.997488 106.298956)
+		(end 167.5 106.801468)
 		(width 0.5)
 		(layer "F.Cu")
@@
 		(width 0.5)
 		(layer "F.Cu")
-		(net 2)
-	)
-	(segment
-		(start 131.669827 96.819827)
-		(end 132.85 98)
-		(width 0.5)
-		(layer "F.Cu")
