File: turret kicad/inf turret.kicad_pcb (KiCad board)
At the start: 2 copper layers, 45 x 45 mm, 27 parts, among them J1 Conn_01x06_Pin, J3 Conn_01x03_Pin, U1 XIAO-ESP32S3

Commit message: add forth pin because i forgot the servo one
Parts:
- removed J3: Conn_01x03_Pin, Connector_PinHeader_2.54mm:PinHeader_1x03_P2.54mm_Vertical
- added J2: Conn_01x04_Pin, Connector_PinHeader_2.54mm:PinHeader_1x04_P2.54mm_Vertical, F.Cu at (143.7, 119.4)
- moved ? 0.57 mm to (161.0, 91.8)
Connections:
- U1 pad 2: unconnected-(U1-PA4_A1_D1-Pad2) -> PWM SERVO
Routing:
- net PWM SERVO: track 0.00 -> 27.8 mm
- net GND: track 65.3 -> 91.9 mm
- net PWM MOTOR: track 23.1 -> 21.5 mm

Commit message: update the design slightly
Parts:
- removed U$30, U$31, U$33 (x2), U$34: MOUNTINGHOLE2.5, Adafruit VL53L4CX:MOUNTINGHOLE_2.5_PLATED
- added ?: , , F.Cu at (157.9, 117.1)
- added ?: , , F.Cu at (133.8, 93.6)
- added ?: , , F.Cu at (157.9, 104.4)
- added ?: , , F.Cu at (137.6, 117.1)
- added ?: , , F.Cu at (137.6, 104.4)
- R5: footprint Resistor_SMD:R_0603_1608Metric -> Resistor_SMD:R_0805_2012Metric
- moved G*** 0.28 mm to (132.8, 104.8)
Routing:
- net +5V: track 156.4 -> 185.9 mm
- net VCC: track 24.0 -> 31.1 mm
- net GND: track 91.9 -> 97.9 mm, vias 11 -> 12
