File: turret kicad/inf turret.kicad_sch (KiCad schematic)
At the start: 7 parts, among them J1 Conn_01x06_Pin, J2 Conn_01x04_Pin, U1 XIAO-ESP32S3

Commit message: update the design slightly
Parts:
- R5: footprint Resistor_SMD:R_0603_1608Metric -> Resistor_SMD:R_0805_2012Metric
Changed lines of the file:
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@@
 			)
 		)
-		(property "Footprint" "Resistor_SMD:R_0603_1608Metric"
+		(property "Footprint" "Resistor_SMD:R_0805_2012Metric"
 			(at 196.85 50.292 90)
 			(effects
